File: hardware_PCB/Main_Board_COYOTE/Main_Board_COYOTE.kicad_sch (KiCad schematic)
At the start: 47 parts, among them J2 Conn_01x05_Pin, J3 Conn_01x05_Pin, J3 FTDI, J4 V+-, J5 MOTOR_PINM1A, J6 MOTOR_PINM1B, J7 MOTOR_PINM1A, J8 MOTOR_PINM1B, Q1 2N7002, SW1 SW_SPST, SW2 START, SW3 START, U1 TA6586, U2 AMS1117-3.3, U2 ESP32-WROOM-32, U4 LM7805_TO220, U5 TA6586

Commit message: Terminados los PCBs
Parts:
- renumbered C12 to C10, C4 to C6, C6 to C7, C7 to C8, C11 to C9, H2 to H1, H1 to H2, H4 to H3, H3 to H4, J4 to J2, J2 to J4, R2 to R1, R4 to R2, R6 to R3, R7 to R4, R1 to R5, R8 to R6, R3 to R7, U4 to U2, U1 to U3, U2 to U4
Other:
- note added: "BUTTON:"
- note added: "CONECTOR:"
- note added: "DRIVER MOTOR TA6586:"
- note added: "ESP32:"
- note added: "HOLE:"
- note added: "LEDS BUZZER:"
- note added: "PROGRAMADOR:"
- note added: "VOLTAGE SUPPLY"
- moved on the sheet: BOOT1, C10, C2, C3, C6, C7, C8, C9, EN1, H1, H2, H3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
