File: hardware_PCB/QRE1113_Line_Sensors_x8/QRE1113_Line_Sensors_x8.kicad_pcb (KiCad board)
At the start: 2 copper layers, 80 x 18 mm, 30 parts, among them J1 Conn_01x05_Pin, J2 Conn_01x05_Pin, U1 QRE1113GR, U2 QRE1113GR, U3 QRE1113GR, U4 QRE1113GR, U5 QRE1113GR, U6 QRE1113GR, U7 QRE1113GR, U8 QRE1113GR

Commit message: Terminados los PCBs
Parts:
- moved J2 5.08 mm to (131.1, 68.8)
- moved J1 5.08 mm to (178.3, 68.8)
Connections:
- J2 pad 4: /OUT_6 -> /OUT_5
- J2 pad 5: /OUT_5 -> /OUT_6
Routing:
- net /OUT_5: track 16.2 -> 26.2 mm
- net /OUT_4: track 12.7 -> 17.8 mm
- net /OUT_1: track 14.9 -> 9.82 mm
- net /OUT_3: track 7.26 -> 11.6 mm
- net /OUT_8: track 13.0 -> 8.83 mm
- net /OUT_7: track 7.33 -> 9.86 mm
- net /OUT_2: track 9.79 -> 7.62 mm
- net /OUT_6: track 9.93 -> 11.8 mm
- net GND: track 46.5 -> 45.0 mm
- net +3V3: track 170.8 -> 171.5 mm
