File: hardware_PCB/QRE1113_Line_Sensors_x8/QRE1113_Line_Sensors_x8.kicad_sch (KiCad schematic)
At the start: 30 parts, among them J1 Conn_01x05_Pin, J2 Conn_01x05_Pin, U1 QRE1113GR, U2 QRE1113GR, U3 QRE1113GR, U4 QRE1113GR, U5 QRE1113GR, U6 QRE1113GR, U7 QRE1113GR, U8 QRE1113GR

Commit message: Terminados los PCBs
Connections:
- net OUT_5: now also J2.4 (Pin_4); no longer J2.5 (Pin_5)
- net OUT_6: now also J2.5 (Pin_5); no longer J2.4 (Pin_4)
Other:
- note added: "CONECTORES:"
- note added: "QRE1113:"
- company: E.E.S.T. Nº5  -> DERTECH - Corporation
Changed lines of the file:
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@@
     (date "2023-07-27")
     (rev "1.0")
-    (company "E.E.S.T. Nº5 ")
+    (company "DERTECH - Corporation")
     (comment 1 "Autor: Mauricio Falcon")
-    (comment 2 "Curso: 7º3º")
   )
   (junction (at 172.2374 85.598) (diameter 0) (color 0 0 0 0)
@@
     (stroke (width 0) (type default))
   )
+  (text "QRE1113:" (at 70.4596 50.7238 0)
+    (effects (font (size 1.651 1.651) (thickness 0.6096) bold) (justify left bottom))
+  )
   (text "CAPACITOR:" (at 197.4596 106.7308 0)
     (effects (font (size 1.651 1.651) (thickness 0.6096) bold) (justify left bottom))
   )
+  (text "CONECTORES:\n" (at 195.5038 50.927 0)
+    (effects (font (size 1.651 1.651) (thickness 0.6096) bold) (justify left bottom))
+  )
   (text "HOLE:" (at 226.187 132.3848 0)
     (effects (font (size 1.651 1.651) (thickness 0.6096) bold) (justify left bottom))
@@
     (effects (font (size 1.27 1.27)) (justify left bottom))
   )
-  (label "OUT_5" (at 215.1126 92.3798 0) (fields_autoplaced)
+  (label "OUT_5" (at 215.1126 89.8398 0) (fields_autoplaced)
     (effects (font (size 1.524 1.524)) (justify left bottom))
   )
@@
     (effects (font (size 1.27 1.27)) (justify left bottom))
   )
-  (label "OUT_6" (at 215.1126 89.8398 0) (fields_autoplaced)
+  (label "OUT_6" (at 215.1126 92.3798 0) (fields_autoplaced)
     (effects (font (size 1.524 1.524)) (justify left bottom))
   )
@@
         )
       )
-    )
-  )
-  (symbol (lib_id "EESTN5-v2:LOGO_ROTULO") (at 259.7404 173.6344 0) (unit 1)
-    (in_bom yes) (on_board yes) (dnp no) (fields_autoplaced)
-    (property "Reference" "#G1" (at 259.7404 179.2732 0)
-      (effects (font (size 1.524 1.524)) hide)
-    )
-    (property "Value" "LOGO_ROTULO" (at 259.7404 167.9956 0)
-      (effects (font (size 1.524 1.524)) hide)
-    )
-    (property "Footprint" "" (at 259.7404 173.6344 0)
-      (effects (font (size 1.524 1.524)) hide)
-    )
-    (property "Datasheet" "" (at 259.7404 173.6344 0)
-      (effects (font (size 1.524 1.524)) hide)
-    )
-    (instances
-      (project "QRE1113_Line_Sensors_x8"
-        (path "/e61bd12c-98c1-486c-9a9e-4493d45b2bcb"
-          (reference "#G1") (unit 1)
-        )
-      )
